Commit message: Final tuning

File: acrobot/acrobot.urdf (robot description, URDF)
Before this commit: robot double_pendulum, 6 links, 5 joints
Joints:
- joint joint1: limit lower=-10000 upper=10000 effort=0 velocity=30 -> lower=-10000 upper=10000 effort=0.15 velocity=50
- joint joint2: limit lower=-10000 upper=10000 effort=0.1 velocity=30 -> lower=-10000 upper=10000 effort=0.15 velocity=50

File: pendubot/pendubot.urdf (robot description, URDF)
Before this commit: robot double_pendulum, 6 links, 5 joints
Links:
- link link1: mass 0.03048177618443695 -> 0.05048177618443695
