Commit message: Updated Pendubot URDF

File: pendubot/pendubot.urdf (robot description, URDF)
Before this commit: robot double_pendulum, 6 links, 5 joints
Links:
- link link1: mass 0.10548177618443695 -> 0.03048177618443695

Commit message: Added Python 3.13 SSQPY extension, reverted Pendubot URDF changes

File: pendubot/pendubot.urdf (robot description, URDF)
Before this commit: robot double_pendulum, 6 links, 5 joints
Links:
- link link1: mass 0.05048177618443695 -> 0.10548177618443695
